Commit message: attempting to distribute sim/viz to other computer

File: src/hexapod_model_description/urdf/hexapod_model.xacro (robot description, xacro)
@@ -12,5 +12,4 @@
         <mesh filename="file://$(find hexapod_model_description)/meshes/base_link.stl" scale="0.001 0.001 0.001"/>
       </geometry>
-      <material name="silver"/>
     </visual>
     <collision>
@@ -32,5 +31,4 @@
         <mesh filename="file://$(find hexapod_model_description)/meshes/leg1_coxa_1.stl" scale="0.001 0.001 0.001"/>
       </geometry>
-      <material name="silver"/>
     </visual>
     <collision>
@@ -52,5 +50,4 @@
         <mesh filename="file://$(find hexapod_model_description)/meshes/leg1_femur_1.stl" scale="0.001 0.001 0.001"/>
       </geometry>
-      <material name="silver"/>
     </visual>
     <collision>
@@ -72,5 +69,4 @@
         <mesh filename="file://$(find hexapod_model_description)/meshes/leg1_tibia_1.stl" scale="0.001 0.001 0.001"/>
       </geometry>
-      <material name="silver"/>
     </visual>
     <collision>
@@ -92,5 +88,4 @@
         <mesh filename="file://$(find hexapod_model_description)/meshes/leg2_coxa_1.stl" scale="0.001 0.001 0.001"/>
       </geometry>
-      <material name="silver"/>
     </visual>
     <collision>
@@ -112,5 +107,4 @@
         <mesh filename="file://$(find hexapod_model_description)/meshes/leg2_femur_1.stl" scale="0.001 0.001 0.001"/>
       </geometry>
-      <material name="silver"/>
     </visual>
     <collision>
@@ -132,5 +126,4 @@
         <mesh filename="file://$(find hexapod_model_description)/meshes/leg2_tibia_1.stl" scale="0.001 0.001 0.001"/>
       </geometry>
-      <material name="silver"/>
     </visual>
     <collision>
@@ -152,5 +145,4 @@
         <mesh filename="file://$(find hexapod_model_description)/meshes/leg3_coxa_1.stl" scale="0.001 0.001 0.001"/>
       </geometry>
-      <material name="silver"/>
     </visual>
     <collision>
@@ -172,5 +164,4 @@
         <mesh filename="file://$(find hexapod_model_description)/meshes/leg3_femur_1.stl" scale="0.001 0.001 0.001"/>
       </geometry>
-      <material name="silver"/>
     </visual>
     <collision>
@@ -192,5 +183,4 @@
         <mesh filename="file://$(find hexapod_model_description)/meshes/leg3_tibia_1.stl" scale="0.001 0.001 0.001"/>
       </geometry>
-      <material name="silver"/>
     </visual>
     <collision>
@@ -212,5 +202,4 @@
         <mesh filename="file://$(find hexapod_model_description)/meshes/leg4_coxa_1.stl" scale="0.001 0.001 0.001"/>
       </geometry>
-      <material name="silver"/>
     </visual>
     <collision>
@@ -232,5 +221,4 @@
         <mesh filename="file://$(find hexapod_model_description)/meshes/leg4_femur_1.stl" scale="0.001 0.001 0.001"/>
       </geometry>
-      <material name="silver"/>
     </visual>
     <collision>
@@ -252,5 +240,4 @@
         <mesh filename="file://$(find hexapod_model_description)/meshes/leg4_tibia_1.stl" scale="0.001 0.001 0.001"/>
       </geometry>
-      <material name="silver"/>
     </visual>
     <collision>
@@ -272,5 +259,4 @@
         <mesh filename="file://$(find hexapod_model_description)/meshes/leg5_coxa_1.stl" scale="0.001 0.001 0.001"/>
       </geometry>
-      <material name="silver"/>
     </visual>
     <collision>
@@ -292,5 +278,4 @@
         <mesh filename="file://$(find hexapod_model_description)/meshes/leg5_femur_1.stl" scale="0.001 0.001 0.001"/>
       </geometry>
-      <material name="silver"/>
     </visual>
     <collision>
@@ -312,5 +297,4 @@
         <mesh filename="file://$(find hexapod_model_description)/meshes/leg5_tibia_1.stl" scale="0.001 0.001 0.001"/>
       </geometry>
-      <material name="silver"/>
     </visual>
     <collision>
@@ -332,5 +316,4 @@
         <mesh filename="file://$(find hexapod_model_description)/meshes/leg6_coxa_1.stl" scale="0.001 0.001 0.001"/>
       </geometry>
-      <material name="silver"/>
     </visual>
     <collision>
@@ -352,5 +335,4 @@
         <mesh filename="file://$(find hexapod_model_description)/meshes/leg6_femur_1.stl" scale="0.001 0.001 0.001"/>
       </geometry>
-      <material name="silver"/>
     </visual>
     <collision>
@@ -372,5 +354,4 @@
         <mesh filename="file://$(find hexapod_model_description)/meshes/leg6_tibia_1.stl" scale="0.001 0.001 0.001"/>
       </geometry>
-      <material name="silver"/>
     </visual>
     <collision>
@@ -392,5 +373,4 @@
         <mesh filename="file://$(find hexapod_model_description)/meshes/neck_1.stl" scale="0.001 0.001 0.001"/>
       </geometry>
-      <material name="silver"/>
     </visual>
     <collision>
@@ -412,5 +392,4 @@
         <mesh filename="file://$(find hexapod_model_description)/meshes/face_1.stl" scale="0.001 0.001 0.001"/>
       </geometry>
-      <material name="silver"/>
     </visual>
     <collision>

Commit message: updated router info

File: src/hexapod_model_description/urdf/hexapod_model.xacro (robot description, xacro)
@@ -1,18 +1,25 @@
 <?xml version="1.0" ?>
 <robot name="hexapod_model" xmlns:xacro="http://www.ros.org/wiki/xacro">
+  <material name="dark_gray">
+    <color rgba="0.3 0.3 0.3 1.0"/>
+  </material>
+  <material name="teal">
+    <color rgba="0.341 0.737 0.753 1.0"/>
+  </material>
   <link name="base_link">
     <inertial>
-      <origin xyz="-0.0026194670129086545 0.000608332751685821 0.039037168945194906" rpy="0 0 0"/>
+      <origin rpy="0 0 0" xyz="-0.0026194670129086545 0.000608332751685821 0.039037168945194906"/>
       <mass value="0.13162148571103816"/>
-      <inertia ixx="0.000549" iyy="0.000616" izz="0.000817" ixy="1e-06" iyz="0.0" ixz="-1e-06"/>
-    </inertial>
-    <visual>
-      <origin xyz="0 0 0" rpy="0 0 0"/>
+      <inertia ixx="0.000549" ixy="1e-06" ixz="-1e-06" iyy="0.000616" iyz="0.0" izz="0.000817"/>
+    </inertial>
+    <visual>
+      <origin rpy="0 0 0" xyz="0 0 0"/>
       <geometry>
         <mesh filename="file://$(find hexapod_model_description)/meshes/base_link.stl" scale="0.001 0.001 0.001"/>
       </geometry>
-    </visual>
-    <collision>
-      <origin xyz="0 0 0" rpy="0 0 0"/>
+      <material name="dark_gray"/>
+    </visual>
+    <collision>
+      <origin rpy="0 0 0" xyz="0 0 0"/>
       <geometry>
         <mesh filename="file://$(find hexapod_model_description)/meshes/base_link.stl" scale="0.001 0.001 0.001"/>
@@ -22,16 +29,17 @@
   <link name="leg1_coxa_1">
     <inertial>
-      <origin xyz="0.02068327294528985 0.0005734513933340138 -0.030108799221667246" rpy="0 0 0"/>
+      <origin rpy="0 0 0" xyz="0.02068327294528985 0.0005734513933340138 -0.030108799221667246"/>
       <mass value="0.055411212779882334"/>
-      <inertia ixx="1.8e-05" iyy="2.7e-05" izz="2.7e-05" ixy="3e-06" iyz="-0.0" ixz="-1e-06"/>
-    </inertial>
-    <visual>
-      <origin xyz="-0.074015 0.054485 -0.072913" rpy="0 0 0"/>
+      <inertia ixx="1.8e-05" ixy="3e-06" ixz="-1e-06" iyy="2.7e-05" iyz="-0.0" izz="2.7e-05"/>
+    </inertial>
+    <visual>
+      <origin rpy="0 0 0" xyz="-0.074015 0.054485 -0.072913"/>
       <geometry>
         <mesh filename="file://$(find hexapod_model_description)/meshes/leg1_coxa_1.stl" scale="0.001 0.001 0.001"/>
       </geometry>
-    </visual>
-    <collision>
-      <origin xyz="-0.074015 0.054485 -0.072913" rpy="0 0 0"/>
+      <material name="teal"/>
+    </visual>
+    <collision>
+      <origin rpy="0 0 0" xyz="-0.074015 0.054485 -0.072913"/>
       <geometry>
         <mesh filename="file://$(find hexapod_model_description)/meshes/leg1_coxa_1.stl" scale="0.001 0.001 0.001"/>
@@ -41,16 +49,17 @@
   <link name="leg1_femur_1">
     <inertial>
-      <origin xyz="0.03542791988760889 -0.02785834312448089 -2.791239019570013e-07" rpy="0 0 0"/>
+      <origin rpy="0 0 0" xyz="0.03542791988760889 -0.02785834312448089 -2.791239019570013e-07"/>
       <mass value="0.01565033360529556"/>
-      <inertia ixx="2.3e-05" iyy="2.2e-05" izz="6e-06" ixy="1e-06" iyz="2e-06" ixz="-1e-06"/>
-    </inertial>
-    <visual>
-      <origin xyz="-0.093074 0.0848 -0.031513" rpy="0 0 0"/>
+      <inertia ixx="2.3e-05" ixy="1e-06" ixz="-1e-06" iyy="2.2e-05" iyz="2e-06" izz="6e-06"/>
+    </inertial>
+    <visual>
+      <origin rpy="0 0 0" xyz="-0.093074 0.0848 -0.031513"/>
       <geometry>
         <mesh filename="file://$(find hexapod_model_description)/meshes/leg1_femur_1.stl" scale="0.001 0.001 0.001"/>
       </geometry>
-    </visual>
-    <collision>
-      <origin xyz="-0.093074 0.0848 -0.031513" rpy="0 0 0"/>
+      <material name="dark_gray"/>
+    </visual>
+    <collision>
+      <origin rpy="0 0 0" xyz="-0.093074 0.0848 -0.031513"/>
       <geometry>
         <mesh filename="file://$(find hexapod_model_description)/meshes/leg1_femur_1.stl" scale="0.001 0.001 0.001"/>
@@ -60,16 +69,17 @@
   <link name="leg1_tibia_1">
     <inertial>
-      <origin xyz="0.015081196994244234 0.02146871541494612 -0.01725662928572464" rpy="0 0 0"/>
+      <origin rpy="0 0 0" xyz="0.015081196994244234 0.02146871541494612 -0.01725662928572464"/>
       <mass value="0.03236606751747676"/>
-      <inertia ixx="2.3e-05" iyy="2.2e-05" izz="5e-06" ixy="-1e-06" iyz="-3e-06" ixz="-1e-06"/>
-    </inertial>
-    <visual>
-      <origin xyz="-0.166798 0.136421 -0.031513" rpy="0 0 0"/>
+      <inertia ixx="2.3e-05" ixy="-1e-06" ixz="-1e-06" iyy="2.2e-05" iyz="-3e-06" izz="5e-06"/>
+    </inertial>
+    <visual>
+      <origin rpy="0 0 0" xyz="-0.166798 0.136421 -0.031513"/>
       <geometry>
         <mesh filename="file://$(find hexapod_model_description)/meshes/leg1_tibia_1.stl" scale="0.001 0.001 0.001"/>
       </geometry>
-    </visual>
-    <collision>
-      <origin xyz="-0.166798 0.136421 -0.031513" rpy="0 0 0"/>
+      <material name="teal"/>
+    </visual>
+    <collision>
+      <origin rpy="0 0 0" xyz="-0.166798 0.136421 -0.031513"/>
       <geometry>
         <mesh filename="file://$(find hexapod_model_description)/meshes/leg1_tibia_1.stl" scale="0.001 0.001 0.001"/>
@@ -79,16 +89,17 @@
   <link name="leg2_coxa_1">
     <inertial>
-      <origin xyz="0.012333292372850486 -0.016614177581995307 -0.030108799221672464" rpy="0 0 0"/>
+      <origin rpy="0 0 0" xyz="0.012333292372850486 -0.016614177581995307 -0.030108799221672464"/>
       <mass value="0.05541121277989177"/>
-      <inertia ixx="2.6e-05" iyy="1.8e-05" izz="2.7e-05" ixy="3e-06" iyz="1e-06" ixz="-0.0"/>
-    </inertial>
-    <visual>
-      <origin xyz="0.001985 0.084485 -0.072913" rpy="0 0 0"/>
+      <inertia ixx="2.6e-05" ixy="3e-06" ixz="-0.0" iyy="1.8e-05" iyz="1e-06" izz="2.7e-05"/>
+    </inertial>
+    <visual>
+      <origin rpy="0 0 0" xyz="0.001985 0.084485 -0.072913"/>
       <geometry>
         <mesh filename="file://$(find hexapod_model_description)/meshes/leg2_coxa_1.stl" scale="0.001 0.001 0.001"/>
       </geometry>
-    </visual>
-    <collision>
-      <origin xyz="0.001985 0.084485 -0.072913" rpy="0 0 0"/>
+      <material name="teal"/>
+    </visual>
+    <collision>
+      <origin rpy="0 0 0" xyz="0.001985 0.084485 -0.072913"/>
       <geometry>
         <mesh filename="file://$(find hexapod_model_description)/meshes/leg2_coxa_1.stl" scale="0.001 0.001 0.001"/>
@@ -98,16 +109,17 @@
   <link name="leg2_femur_1">
     <inertial>
-      <origin xyz="-0.0025002890984096374 -0.04419164973443521 -0.008492801491495987" rpy="0 0 0"/>
+      <origin rpy="0 0 0" xyz="-0.0025002890984096374 -0.04419164973443521 -0.008492801491495987"/>
       <mass value="0.015650333605295393"/>
-      <inertia ixx="2.3e-05" iyy="2.2e-05" izz="6e-06" ixy="1e-06" iyz="2e-06" ixz="-1e-06"/>
-    </inertial>
-    <visual>
-      <origin xyz="0.015885 0.117485 -0.031513" rpy="0 0 0"/>
+      <inertia ixx="2.3e-05" ixy="1e-06" ixz="-1e-06" iyy="2.2e-05" iyz="2e-06" izz="6e-06"/>
+    </inertial>
+    <visual>
+      <origin rpy="0 0 0" xyz="0.015885 0.117485 -0.031513"/>
       <geometry>
         <mesh filename="file://$(find hexapod_model_description)/meshes/leg2_femur_1.stl" scale="0.001 0.001 0.001"/>
       </geometry>
-    </visual>
-    <collision>
-      <origin xyz="0.015885 0.117485 -0.031513" rpy="0 0 0"/>
+      <material name="dark_gray"/>
+    </visual>
+    <collision>
+      <origin rpy="0 0 0" xyz="0.015885 0.117485 -0.031513"/>
       <geometry>
         <mesh filename="file://$(find hexapod_model_description)/meshes/leg2_femur_1.stl" scale="0.001 0.001 0.001"/>
@@ -117,16 +129,17 @@
   <link name="leg2_tibia_1">
     <inertial>
-      <origin xyz="0.02623657202447643 0.0032175056252809753 -0.016954107546123608" rpy="0 0 0"/>
+      <origin rpy="0 0 0" xyz="0.02623657202447643 0.0032175056252809753 -0.016954107546123608"/>
       <mass value="0.032366066740945575"/>
-      <inertia ixx="2.1e-05" iyy="2.3e-05" izz="6e-06" ixy="1e-06" iyz="3e-06" ixz="-3e-06"/>
-    </inertial>
-    <visual>
-      <origin xyz="0.015885 0.205868 -0.014528" rpy="0 0 0"/>
+      <inertia ixx="2.1e-05" ixy="1e-06" ixz="-3e-06" iyy="2.3e-05" iyz="3e-06" izz="6e-06"/>
+    </inertial>
+    <visual>
+      <origin rpy="0 0 0" xyz="0.015885 0.205868 -0.014528"/>
       <geometry>
         <mesh filename="file://$(find hexapod_model_description)/meshes/leg2_tibia_1.stl" scale="0.001 0.001 0.001"/>
       </geometry>
-    </visual>
-    <collision>
-      <origin xyz="0.015885 0.205868 -0.014528" rpy="0 0 0"/>
+      <material name="teal"/>
+    </visual>
+    <collision>
+      <origin rpy="0 0 0" xyz="0.015885 0.205868 -0.014528"/>
       <geometry>
         <mesh filename="file://$(find hexapod_model_description)/meshes/leg2_tibia_1.stl" scale="0.001 0.001 0.001"/>
@@ -136,16 +149,17 @@
   <link name="leg3_coxa_1">
     <inertial>
-      <origin xyz="-0.004799395854957936 -0.020127553637971148 -0.030108799221667412" rpy="0 0 0"/>
+      <origin rpy="0 0 0" xyz="-0.004799395854957936 -0.020127553637971148 -0.030108799221667412"/>
       <mass value="0.055411212779882306"/>
-      <inertia ixx="2.5e-05" iyy="2e-05" izz="2.7e-05" ixy="-5e-06" iyz="1e-06" ixz="0.0"/>
-    </inertial>
-    <visual>
-      <origin xyz="0.077985 0.054485 -0.072913" rpy="0 0 0"/>
+      <inertia ixx="2.5e-05" ixy="-5e-06" ixz="0.0" iyy="2e-05" iyz="1e-06" izz="2.7e-05"/>
+    </inertial>
+    <visual>
+      <origin rpy="0 0 0" xyz="0.077985 0.054485 -0.072913"/>
       <geometry>
         <mesh filename="file://$(find hexapod_model_description)/meshes/leg3_coxa_1.stl" scale="0.001 0.001 0.001"/>
       </geometry>
-    </visual>
-    <collision>
-      <origin xyz="0.077985 0.054485 -0.072913" rpy="0 0 0"/>
+      <material name="teal"/>
+    </visual>
+    <collision>
+      <origin rpy="0 0 0" xyz="0.077985 0.054485 -0.072913"/>
       <geometry>
         <mesh filename="file://$(find hexapod_model_description)/meshes/leg3_coxa_1.stl" scale="0.001 0.001 0.001"/>
@@ -155,16 +169,17 @@
   <link name="leg3_femur_1">
     <inertial>
-      <origin xyz="-0.036078469514005895 -0.027010579982379296 -2.791239018945513e-07" rpy="0 0 0"/>
+      <origin rpy="0 0 0" xyz="-0.036078469514005895 -0.027010579982379296 -2.791239018945513e-07"/>
       <mass value="0.01565033360529561"/>
-      <inertia ixx="2.3e-05" iyy="2.2e-05" izz="6e-06" ixy="1e-06" iyz="2e-06" ixz="-1e-06"/>
-    </inertial>
-    <visual>
-      <origin xyz="0.1122 0.065049 -0.031513" rpy="0 0 0"/>
+      <inertia ixx="2.3e-05" ixy="1e-06" ixz="-1e-06" iyy="2.2e-05" iyz="2e-06" izz="6e-06"/>
+    </inertial>
+    <visual>
+      <origin rpy="0 0 0" xyz="0.1122 0.065049 -0.031513"/>
       <geometry>
         <mesh filename="file://$(find hexapod_model_description)/meshes/leg3_femur_1.stl" scale="0.001 0.001 0.001"/>
       </geometry>
-    </visual>
-    <collision>
-      <origin xyz="0.1122 0.065049 -0.031513" rpy="0 0 0"/>
+      <material name="dark_gray"/>
+    </visual>
+    <collision>
+      <origin rpy="0 0 0" xyz="0.1122 0.065049 -0.031513"/>
       <geometry>
         <mesh filename="file://$(find hexapod_model_description)/meshes/leg3_femur_1.stl" scale="0.001 0.001 0.001"/>
@@ -174,16 +189,17 @@
   <link name="leg3_tibia_1">
     <inertial>
-      <origin xyz="0.016834697294396933 -0.02012435473824882 -0.017256629587411518" rpy="0 0 0"/>
+      <origin rpy="0 0 0" xyz="0.016834697294396933 -0.02012435473824882 -0.017256629587411518"/>
       <mass value="0.0323660675174863"/>
-      <inertia ixx="2.2e-05" iyy="2.2e-05" izz="5e-06" ixy="1e-06" iyz="2e-06" ixz="-2e-06"/>
-    </inertial>
-    <visual>
-      <origin xyz="0.181144 0.1229 -0.031513" rpy="0 0 0"/>
+      <inertia ixx="2.2e-05" ixy="1e-06" ixz="-2e-06" iyy="2.2e-05" iyz="2e-06" izz="5e-06"/>
+    </inertial>
+    <visual>
+      <origin rpy="0 0 0" xyz="0.181144 0.1229 -0.031513"/>
       <geometry>
         <mesh filename="file://$(find hexapod_model_description)/meshes/leg3_tibia_1.stl" scale="0.001 0.001 0.001"/>
       </geometry>
-    </visual>
-    <collision>
-      <origin xyz="0.181144 0.1229 -0.031513" rpy="0 0 0"/>
+      <material name="teal"/>
+    </visual>
+    <collision>
+      <origin rpy="0 0 0" xyz="0.181144 0.1229 -0.031513"/>
       <geometry>
         <mesh filename="file://$(find hexapod_model_description)/meshes/leg3_tibia_1.stl" scale="0.001 0.001 0.001"/>
@@ -193,16 +209,17 @@
   <link name="leg4_coxa_1">
     <inertial>
-      <origin xyz="-0.004799396098101663 0.020126991093514547 -0.030108799033593925" rpy="0 0 0"/>
+      <origin rpy="0 0 0" xyz="-0.004799396098101663 0.020126991093514547 -0.030108799033593925"/>
       <mass value="0.05541121277988202"/>
-      <inertia ixx="2.5e-05" iyy="2e-05" izz="2.7e-05" ixy="5e-06" iyz="-1e-06" ixz="0.0"/>
-    </inertial>
-    <visual>
-      <origin xyz="0.077985 -0.055515 -0.072913" rpy="0 0 0"/>
+      <inertia ixx="2.5e-05" ixy="5e-06" ixz="0.0" iyy="2e-05" iyz="-1e-06" izz="2.7e-05"/>
+    </inertial>
+    <visual>
+      <origin rpy="0 0 0" xyz="0.077985 -0.055515 -0.072913"/>
       <geometry>
         <mesh filename="file://$(find hexapod_model_description)/meshes/leg4_coxa_1.stl" scale="0.001 0.001 0.001"/>
       </geometry>
-    </visual>
-    <collision>
-      <origin xyz="0.077985 -0.055515 -0.072913" rpy="0 0 0"/>
+      <material name="teal"/>
+    </visual>
+    <collision>
+      <origin rpy="0 0 0" xyz="0.077985 -0.055515 -0.072913"/>
       <geometry>
         <mesh filename="file://$(find hexapod_model_description)/meshes/leg4_coxa_1.stl" scale="0.001 0.001 0.001"/>
@@ -212,16 +229,17 @@
   <link name="leg4_femur_1">
     <inertial>
-      <origin xyz="-0.03607846956725638 0.02701001794357151 -2.78240923724804e-07" rpy="0 0 0"/>
+      <origin rpy="0 0 0" xyz="-0.03607846956725638 0.02701001794357151 -2.78240923724804e-07"/>
       <mass value="0.015650333605295472"/>
-      <inertia ixx="2.3e-05" iyy="2.2e-05" izz="6e-06" ixy="1e-06" iyz="2e-06" ixz="-1e-06"/>
-    </inertial>
-    <visual>
-      <origin xyz="0.1122 -0.066079 -0.031513" rpy="0 0 0"/>
+      <inertia ixx="2.3e-05" ixy="1e-06" ixz="-1e-06" iyy="2.2e-05" iyz="2e-06" izz="6e-06"/>
+    </inertial>
+    <visual>
+      <origin rpy="0 0 0" xyz="0.1122 -0.066079 -0.031513"/>
       <geometry>
         <mesh filename="file://$(find hexapod_model_description)/meshes/leg4_femur_1.stl" scale="0.001 0.001 0.001"/>
       </geometry>
-    </visual>
-    <collision>
-      <origin xyz="0.1122 -0.066079 -0.031513" rpy="0 0 0"/>
+      <material name="dark_gray"/>
+    </visual>
+    <collision>
+      <origin rpy="0 0 0" xyz="0.1122 -0.066079 -0.031513"/>
       <geometry>
         <mesh filename="file://$(find hexapod_model_description)/meshes/leg4_femur_1.stl" scale="0.001 0.001 0.001"/>
@@ -231,16 +249,17 @@
   <link name="leg4_tibia_1">
     <inertial>
-      <origin xyz="0.016834697878780613 0.020123792830575096 -0.01725662819463489" rpy="0 0 0"/>
+      <origin rpy="0 0 0" xyz="0.016834697878780613 0.020123792830575096 -0.01725662819463489"/>
       <mass value="0.03236606751747625"/>
-      <inertia ixx="2.2e-05" iyy="2.2e-05" izz="5e-06" ixy="-1e-06" iyz="-2e-06" ixz="-2e-06"/>
-    </inertial>
-    <visual>
-      <origin xyz="0.181144 -0.12393 -0.031513" rpy="0 0 0"/>
+      <inertia ixx="2.2e-05" ixy="-1e-06" ixz="-2e-06" iyy="2.2e-05" iyz="-2e-06" izz="5e-06"/>
+    </inertial>
+    <visual>
+      <origin rpy="0 0 0" xyz="0.181144 -0.12393 -0.031513"/>
       <geometry>
         <mesh filename="file://$(find hexapod_model_description)/meshes/leg4_tibia_1.stl" scale="0.001 0.001 0.001"/>
       </geometry>
-    </visual>
-    <collision>
-      <origin xyz="0.181144 -0.12393 -0.031513" rpy="0 0 0"/>
+      <material name="teal"/>
+    </visual>
+    <collision>
+      <origin rpy="0 0 0" xyz="0.181144 -0.12393 -0.031513"/>
       <geometry>
         <mesh filename="file://$(find hexapod_model_description)/meshes/leg4_tibia_1.stl" scale="0.001 0.001 0.001"/>
@@ -250,16 +269,17 @@
   <link name="leg5_coxa_1">
     <inertial>
-      <origin xyz="0.01233329237284984 0.01661361515093593 -0.030108799033599393" rpy="0 0 0"/>
+      <origin rpy="0 0 0" xyz="0.01233329237284984 0.01661361515093593 -0.030108799033599393"/>
       <mass value="0.05541121277989181"/>
-      <inertia ixx="2.6e-05" iyy="1.8e-05" izz="2.7e-05" ixy="-3e-06" iyz="-1e-06" ixz="-0.0"/>
-    </inertial>
-    <visual>
-      <origin xyz="0.001985 -0.085515 -0.072913" rpy="0 0 0"/>
+      <inertia ixx="2.6e-05" ixy="-3e-06" ixz="-0.0" iyy="1.8e-05" iyz="-1e-06" izz="2.7e-05"/>
+    </inertial>
+    <visual>
+      <origin rpy="0 0 0" xyz="0.001985 -0.085515 -0.072913"/>
       <geometry>
         <mesh filename="file://$(find hexapod_model_description)/meshes/leg5_coxa_1.stl" scale="0.001 0.001 0.001"/>
       </geometry>
-    </visual>
-    <collision>
-      <origin xyz="0.001985 -0.085515 -0.072913" rpy="0 0 0"/>
+      <material name="teal"/>
+    </visual>
+    <collision>
+      <origin rpy="0 0 0" xyz="0.001985 -0.085515 -0.072913"/>
       <geometry>
         <mesh filename="file://$(find hexapod_model_description)/meshes/leg5_coxa_1.stl" scale="0.001 0.001 0.001"/>
@@ -269,16 +289,17 @@
   <link name="leg5_femur_1">
     <inertial>
-      <origin xyz="-0.0025002885936068545 0.04499443236815963 0.0006894733466853292" rpy="0 0 0"/>
+      <origin rpy="0 0 0" xyz="-0.0025002885936068545 0.04499443236815963 0.0006894733466853292"/>
       <mass value="0.01565033360529512"/>
-      <inertia ixx="2.3e-05" iyy="2.2e-05" izz="6e-06" ixy="1e-06" iyz="2e-06" ixz="-1e-06"/>
-    </inertial>
-    <visual>
-      <origin xyz="0.015885 -0.118515 -0.031513" rpy="0 0 0"/>
+      <inertia ixx="2.3e-05" ixy="1e-06" ixz="-1e-06" iyy="2.2e-05" iyz="2e-06" izz="6e-06"/>
+    </inertial>
+    <visual>
+      <origin rpy="0 0 0" xyz="0.015885 -0.118515 -0.031513"/>
       <geometry>
         <mesh filename="file://$(find hexapod_model_description)/meshes/leg5_femur_1.stl" scale="0.001 0.001 0.001"/>
       </geometry>
-    </visual>
-    <collision>
-      <origin xyz="0.015885 -0.118515 -0.031513" rpy="0 0 0"/>
+      <material name="dark_gray"/>
+    </visual>
+    <collision>
+      <origin rpy="0 0 0" xyz="0.015885 -0.118515 -0.031513"/>
       <geometry>
         <mesh filename="file://$(find hexapod_model_description)/meshes/leg5_femur_1.stl" scale="0.001 0.001 0.001"/>
@@ -288,16 +309,17 @@
   <link name="leg5_tibia_1">
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